Commit message: wrong package referenced in urdf

File: urdf/accessories.urdf.xacro (robot description, xacro)
@@ -10,15 +10,15 @@
       <visual>
         <geometry>
-          <mesh filename="package://spot_description/meshes/pack_top.dae"/>
+          <mesh filename="package://spot_gazebo_sim/meshes/pack_top.dae"/>
         </geometry>
       </visual>
       <visual>
         <geometry>
-          <mesh filename="package://spot_description/meshes/pack_body.dae"/>
+          <mesh filename="package://spot_gazebo_sim/meshes/pack_body.dae"/>
         </geometry>
       </visual>
       <collision>
         <geometry>
-          <mesh filename="package://spot_description/meshes/pack_body.dae"/>
+          <mesh filename="package://spot_gazebo_sim/meshes/pack_body.dae"/>
         </geometry>
       </collision>
@@ -34,10 +34,10 @@
       <visual>
         <geometry>
-          <mesh filename="package://spot_description/meshes/lidar_mount.dae"/>
+          <mesh filename="package://spot_gazebo_sim/meshes/lidar_mount.dae"/>
         </geometry>
       </visual>
       <collision>
         <geometry>
-          <mesh filename="package://spot_description/meshes/lidar_mount_collision.stl"/>
+          <mesh filename="package://spot_gazebo_sim/meshes/lidar_mount_collision.stl"/>
         </geometry>
       </collision>
@@ -52,10 +52,10 @@
         <visual>
           <geometry>
-            <mesh filename="package://spot_description/meshes/velo.dae"/>
+            <mesh filename="package://spot_gazebo_sim/meshes/velo.dae"/>
           </geometry>
         </visual>
         <collision>
           <geometry>
-            <mesh filename="package://spot_description/meshes/velo_collision.stl"/>
+            <mesh filename="package://spot_gazebo_sim/meshes/velo_collision.stl"/>
           </geometry>
         </collision>

File: urdf/spot.urdf.xacro (robot description, xacro)
@@ -4,10 +4,10 @@
         <visual>
             <geometry>
-                <mesh filename="package://spot_description/meshes/body.dae" />
-            </geometry>
-        </visual>
-        <collision>
-            <geometry>
-                <mesh filename="package://spot_description/meshes/body_collision.stl" />
+                <mesh filename="package://spot_gazebo_sim/meshes/body.dae" />
+            </geometry>
+        </visual>
+        <collision>
+            <geometry>
+                <mesh filename="package://spot_gazebo_sim/meshes/body_collision.stl" />
             </geometry>
         </collision>
@@ -34,10 +34,10 @@
         <visual>
             <geometry>
-                <mesh filename="package://spot_description/meshes/front_left_hip.dae" />
-            </geometry>
-        </visual>
-        <collision>
-            <geometry>
-                <mesh filename="package://spot_description/meshes/front_left_hip_collision.stl" />
+                <mesh filename="package://spot_gazebo_sim/meshes/front_left_hip.dae" />
+            </geometry>
+        </visual>
+        <collision>
+            <geometry>
+                <mesh filename="package://spot_gazebo_sim/meshes/front_left_hip_collision.stl" />
             </geometry>
         </collision>
@@ -53,10 +53,10 @@
         <visual>
             <geometry>
-                <mesh filename="package://spot_description/meshes/front_left_upper_leg.dae" />
-            </geometry>
-        </visual>
-        <collision>
-            <geometry>
-                <mesh filename="package://spot_description/meshes/front_left_upper_leg_collision.stl" />
+                <mesh filename="package://spot_gazebo_sim/meshes/front_left_upper_leg.dae" />
+            </geometry>
+        </visual>
+        <collision>
+            <geometry>
+                <mesh filename="package://spot_gazebo_sim/meshes/front_left_upper_leg_collision.stl" />
             </geometry>
         </collision>
@@ -72,10 +72,10 @@
         <visual>
             <geometry>
-                <mesh filename="package://spot_description/meshes/front_left_lower_leg.dae" />
-            </geometry>
-        </visual>
-        <collision>
-            <geometry>
-                <mesh filename="package://spot_description/meshes/front_left_lower_leg_collision.stl" />
+                <mesh filename="package://spot_gazebo_sim/meshes/front_left_lower_leg.dae" />
+            </geometry>
+        </visual>
+        <collision>
+            <geometry>
+                <mesh filename="package://spot_gazebo_sim/meshes/front_left_lower_leg_collision.stl" />
             </geometry>
         </collision>
@@ -91,10 +91,10 @@
         <visual>
             <geometry>
-                <mesh filename="package://spot_description/meshes/front_right_hip.dae" />
-            </geometry>
-        </visual>
-        <collision>
-            <geometry>
-                <mesh filename="package://spot_description/meshes/front_right_hip_collision.stl" />
+                <mesh filename="package://spot_gazebo_sim/meshes/front_right_hip.dae" />
+            </geometry>
+        </visual>
+        <collision>
+            <geometry>
+                <mesh filename="package://spot_gazebo_sim/meshes/front_right_hip_collision.stl" />
             </geometry>
         </collision>
@@ -110,10 +110,10 @@
         <visual>
             <geometry>
-                <mesh filename="package://spot_description/meshes/front_right_upper_leg.dae" />
-            </geometry>
-        </visual>
-        <collision>
-            <geometry>
-                <mesh filename="package://spot_description/meshes/front_right_upper_leg_collision.stl" />
+                <mesh filename="package://spot_gazebo_sim/meshes/front_right_upper_leg.dae" />
+            </geometry>
+        </visual>
+        <collision>
+            <geometry>
+                <mesh filename="package://spot_gazebo_sim/meshes/front_right_upper_leg_collision.stl" />
             </geometry>
         </collision>
@@ -129,10 +129,10 @@
         <visual>
             <geometry>
-                <mesh filename="package://spot_description/meshes/front_right_lower_leg.dae" />
-            </geometry>
-        </visual>
-        <collision>
-            <geometry>
-                <mesh filename="package://spot_description/meshes/front_right_lower_leg_collision.stl" />
+                <mesh filename="package://spot_gazebo_sim/meshes/front_right_lower_leg.dae" />
+            </geometry>
+        </visual>
+        <collision>
+            <geometry>
+                <mesh filename="package://spot_gazebo_sim/meshes/front_right_lower_leg_collision.stl" />
             </geometry>
         </collision>
@@ -148,10 +148,10 @@
         <visual>
             <geometry>
-                <mesh filename="package://spot_description/meshes/rear_left_hip.dae" />
-            </geometry>
-        </visual>
-        <collision>
-            <geometry>
-                <mesh filename="package://spot_description/meshes/rear_left_hip_collision.stl" />
+                <mesh filename="package://spot_gazebo_sim/meshes/rear_left_hip.dae" />
+            </geometry>
+        </visual>
+        <collision>
+            <geometry>
+                <mesh filename="package://spot_gazebo_sim/meshes/rear_left_hip_collision.stl" />
             </geometry>
         </collision>
@@ -167,10 +167,10 @@
         <visual>
             <geometry>
-                <mesh filename="package://spot_description/meshes/rear_left_upper_leg.dae" />
-            </geometry>
-        </visual>
-        <collision>
-            <geometry>
-                <mesh filename="package://spot_description/meshes/rear_left_upper_leg_collision.stl" />
+                <mesh filename="package://spot_gazebo_sim/meshes/rear_left_upper_leg.dae" />
+            </geometry>
+        </visual>
+        <collision>
+            <geometry>
+                <mesh filename="package://spot_gazebo_sim/meshes/rear_left_upper_leg_collision.stl" />
             </geometry>
         </collision>
@@ -186,10 +186,10 @@
         <visual>
             <geometry>
-                <mesh filename="package://spot_description/meshes/rear_left_lower_leg.dae" />
-            </geometry>
-        </visual>
-        <collision>
-            <geometry>
-                <mesh filename="package://spot_description/meshes/rear_left_lower_leg_collision.stl" />
+                <mesh filename="package://spot_gazebo_sim/meshes/rear_left_lower_leg.dae" />
+            </geometry>
+        </visual>
+        <collision>
+            <geometry>
+                <mesh filename="package://spot_gazebo_sim/meshes/rear_left_lower_leg_collision.stl" />
             </geometry>
         </collision>
@@ -205,10 +205,10 @@
         <visual>
             <geometry>
-                <mesh filename="package://spot_description/meshes/rear_right_hip.dae" />
-            </geometry>
-        </visual>
-        <collision>
-            <geometry>
-                <mesh filename="package://spot_description/meshes/rear_right_hip_collision.stl" />
+                <mesh filename="package://spot_gazebo_sim/meshes/rear_right_hip.dae" />
+            </geometry>
+        </visual>
+        <collision>
+            <geometry>
+                <mesh filename="package://spot_gazebo_sim/meshes/rear_right_hip_collision.stl" />
             </geometry>
         </collision>
@@ -224,10 +224,10 @@
         <visual>
             <geometry>
-                <mesh filename="package://spot_description/meshes/rear_right_upper_leg.dae" />
-            </geometry>
-        </visual>
-        <collision>
-            <geometry>
-                <mesh filename="package://spot_description/meshes/rear_right_upper_leg_collision.stl" />
+                <mesh filename="package://spot_gazebo_sim/meshes/rear_right_upper_leg.dae" />
+            </geometry>
+        </visual>
+        <collision>
+            <geometry>
+                <mesh filename="package://spot_gazebo_sim/meshes/rear_right_upper_leg_collision.stl" />
             </geometry>
         </collision>
@@ -243,10 +243,10 @@
         <visual>
             <geometry>
-                <mesh filename="package://spot_description/meshes/rear_right_lower_leg.dae" />
-            </geometry>
-        </visual>
-        <collision>
-            <geometry>
-                <mesh filename="package://spot_description/meshes/rear_right_lower_leg_collision.stl" />
+                <mesh filename="package://spot_gazebo_sim/meshes/rear_right_lower_leg.dae" />
+            </geometry>
+        </visual>
+        <collision>
+            <geometry>
+                <mesh filename="package://spot_gazebo_sim/meshes/rear_right_lower_leg_collision.stl" />
             </geometry>
         </collision>
@@ -260,4 +260,4 @@
     </joint>
     <!-- Standard accessories. -->
-    <xacro:include filename="$(find spot_description)/urdf/accessories.urdf.xacro" />
+    <xacro:include filename="$(find spot_gazebo_sim)/urdf/accessories.urdf.xacro" />
 </robot>
