Commit message: First working version of Spot, controled through ROS Control.

File: urdf/spot.urdf.xacro (robot description, xacro)
@@ -12,10 +12,14 @@
             </geometry>
         </collision>
+        <inertial>
+             <mass value="16.25" />
+             <inertia  ixx="0.085" ixy="0.0"  ixz="0.0"  iyy="1.045"  iyz="0.0"  izz="1.042" />
+    	</inertial>
     </link>
     <link name="base_link"/>
     <joint name="base_link_joint" type="fixed">
         <origin xyz="0 0 0" rpy="0 0 0" />
-        <parent link="body" />
-        <child link="base_link" />
+        <parent link="base_link" />
+        <child link="body" />
     </joint>
     <link name="front_rail"/>
@@ -42,4 +46,8 @@
             </geometry>
         </collision>
+        <inertial>
+            <mass value="1.5" />
+    	    <inertia  ixx="0.0605" ixy="0.0"  ixz="0.0"  iyy="0.0"  iyz="0.0"  izz="0.0" />
+    	</inertial>
     </link>
     <joint name="front_left_hip_x" type="revolute">
@@ -48,6 +56,17 @@
         <parent link="body" />
         <child link="front_left_hip" />
+	    <dynamics damping="0.1" friction="0.1"/>
         <limit effort="1000" velocity="1000.00" lower="-0.78539816339744827899" upper="0.78539816339744827899" />
     </joint>
+    <transmission name="front_left_hip_x_trans">
+	  <type>transmission_interface/SimpleTransmission</type>
+	  <joint name="front_left_hip_x">
+          	<hardwareInterface>hardware_interface/EffortJointInterface</hardwareInterface>
+          </joint>
+	  <actuator name="front_left_hip_x">
+          	<mechanicalReduction>50</mechanicalReduction>
+          	<hardwareInterface>hardware_interface/EffortJointInterface</hardwareInterface>
+	  </actuator>
+    </transmission>
     <link name="front_left_upper_leg">
         <visual>
@@ -61,4 +80,8 @@
             </geometry>
         </collision>
+        <inertial>
+            <mass value="1.5" />
+    	    <inertia  ixx="0.0" ixy="0.0"  ixz="0.0"  iyy="0.05"  iyz="0.0"  izz="0.0" />
+    	</inertial>
     </link>
     <joint name="front_left_hip_y" type="revolute">
@@ -67,6 +90,17 @@
         <parent link="front_left_hip" />
         <child link="front_left_upper_leg" />
+	    <dynamics damping="0.1" friction="0.1"/>
         <limit effort="1000" velocity="1000.00" lower="-0.89884456477707963539" upper="2.2951079663725435509" />
     </joint>
+    <transmission name="front_left_hip_y_trans">
+	  <type>transmission_interface/SimpleTransmission</type>
+	  <joint name="front_left_hip_y">
+          	<hardwareInterface>hardware_interface/EffortJointInterface</hardwareInterface>
+          </joint>
+	  <actuator name="front_left_hip_y">
+          	<mechanicalReduction>50</mechanicalReduction>
+          	<hardwareInterface>hardware_interface/EffortJointInterface</hardwareInterface>
+	  </actuator>
+    </transmission>
     <link name="front_left_lower_leg">
         <visual>
@@ -80,4 +114,8 @@
             </geometry>
         </collision>
+        <inertial>right
+            <mass value="1.0" />
+    	    <inertia  ixx="0.0" ixy="0.0"  ixz="0.0"  iyy="0.045"  iyz="0.0"  izz="0.0" />
+    	</inertial>
     </link>
     <joint name="front_left_knee" type="revolute">
@@ -86,6 +124,30 @@
         <parent link="front_left_upper_leg" />
         <child link="front_left_lower_leg" />
+        <dynamics damping="0.1" friction="0.1"/>
         <limit effort="1000" velocity="1000.00" lower="-2.7929" upper="-0.254801" />
     </joint>
+    <!-- Optional Contact Sensor (SoftServeSAG) -->
+    <gazebo reference="front_left_lower_leg">
+        <sensor name="front_left_lower_leg_contactsensor_sensor" type="contact">
+        <always_on>true</always_on>
+        <contact>
+            <collision>front_left_lower_leg_fixed_joint_lump__front_bump_sensor_collision</collision>
+        </contact>
+        <plugin filename="libgazebo_ros_bumper.so" name="front_left_lower_leg_plugin">
+            <bumperTopicName>front_left_lower_leg_contact</bumperTopicName>
+            <frameName>front_left_lower_leg</frameName>
+        </plugin>
+        </sensor>
+    </gazebo>
+    <transmission name="front_left_knee_trans">
+	  <type>transmission_interface/SimpleTransmission</type>
+	  <joint name="front_left_knee">
+          	<hardwareInterface>hardware_interface/EffortJointInterface</hardwareInterface>
+          </joint>
+	  <actuator name="front_left_knee">
+          	<mechanicalReduction>50</mechanicalReduction>
+          	<hardwareInterface>hardware_interface/EffortJointInterface</hardwareInterface>
+	  </actuator>
+    </transmission>
     <link name="front_right_hip">
         <visual>
@@ -99,4 +161,8 @@
             </geometry>
         </collision>
+        <inertial>
+            <mass value="1.5" />
+    	    <inertia  ixx="0.0605" ixy="0.0"  ixz="0.0"  iyy="0.0"  iyz="0.0"  izz="0.0" />
+    	</inertial>
     </link>
     <joint name="front_right_hip_x" type="revolute">
@@ -105,6 +171,17 @@
         <parent link="body" />
         <child link="front_right_hip" />
+        <dynamics damping="0.1" friction="0.1"/>
         <limit effort="1000" velocity="1000.00" lower="-0.78539816339744827899" upper="0.78539816339744827899" />
     </joint>
+    <transmission name="front_right_hip_x_trans">
+	  <type>transmission_interface/SimpleTransmission</type>
+	  <joint name="front_right_hip_x">
+          	<hardwareInterface>hardware_interface/EffortJointInterface</hardwareInterface>
+          </joint>
+	  <actuator name="front_right_hip_x">
+          	<mechanicalReduction>50</mechanicalReduction>
+          	<hardwareInterface>hardware_interface/EffortJointInterface</hardwareInterface>
+	  </actuator>
+    </transmission>
     <link name="front_right_upper_leg">
         <visual>
@@ -118,4 +195,8 @@
             </geometry>
         </collision>
+        <inertial>
+            <mass value="1.5" />
+    	    <inertia  ixx="0.0" ixy="0.0"  ixz="0.0"  iyy="0.05"  iyz="0.0"  izz="0.0" />
+    	</inertial>
     </link>
     <joint name="front_right_hip_y" type="revolute">
@@ -124,6 +205,17 @@
         <parent link="front_right_hip" />
         <child link="front_right_upper_leg" />
+        <dynamics damping="0.1" friction="0.1"/>
         <limit effort="1000" velocity="1000.00" lower="-0.89884456477707963539" upper="2.2951079663725435509" />
     </joint>
+    <transmission name="front_right_hip_y_trans">
+	  <type>transmission_interface/SimpleTransmission</type>
+	  <joint name="front_right_hip_y">
+          	<hardwareInterface>hardware_interface/EffortJointInterface</hardwareInterface>
+          </joint>
+	  <actuator name="front_right_hip_y">
+          	<mechanicalReduction>50</mechanicalReduction>
+          	<hardwareInterface>hardware_interface/EffortJointInterface</hardwareInterface>
+	  </actuator>
+    </transmission>
     <link name="front_right_lower_leg">
         <visual>
@@ -137,4 +229,8 @@
             </geometry>
         </collision>
+        <inertial>
+            <mass value="1.0" />
+    	    <inertia  ixx="0.0" ixy="0.0"  ixz="0.0"  iyy="0.045"  iyz="0.0"  izz="0.0" />
+    	</inertial>
     </link>
     <joint name="front_right_knee" type="revolute">
@@ -143,6 +239,30 @@
         <parent link="front_right_upper_leg" />
         <child link="front_right_lower_leg" />
+        <dynamics damping="0.1" friction="0.1"/>
         <limit effort="1000" velocity="1000.00" lower="-2.7929" upper="-0.247563" />
     </joint>
+    <!-- Optional Contact Sensor (SoftserveSAG)-->
+    <gazebo reference="front_right_lower_leg">
+        <sensor name="front_right_lower_leg_contactsensor_sensor" type="contact">
+        <always_on>true</always_on>
+        <contact>
+            <collision>front_right_lower_leg_fixed_joint_lump__front_bump_sensor_collision</collision>
+        </contact>
+        <plugin filename="libgazebo_ros_bumper.so" name="front_right_lower_leg_plugin">
+            <bumperTopicName>front_right_lower_leg_contact</bumperTopicName>
+            <frameName>front_right_lower_leg</frameName>
+        </plugin>
+        </sensor>
+    </gazebo>
+    <transmission name="front_right_knee_trans">
+	  <type>transmission_interface/SimpleTransmission</type>
+	  <joint name="front_right_knee">
+          	<hardwareInterface>hardware_interface/EffortJointInterface</hardwareInterface>
+          </joint>
+	  <actuator name="front_right_knee">
+          	<mechanicalReduction>50</mechanicalReduction>
+          	<hardwareInterface>hardware_interface/EffortJointInterface</hardwareInterface>
+	  </actuator>
+    </transmission>
     <link name="rear_left_hip">
         <visual>
@@ -156,4 +276,8 @@
             </geometry>
         </collision>
+        <inertial>
+            <mass value="1.5" />
+    	    <inertia  ixx="0.0605" ixy="0.0"  ixz="0.0"  iyy="0.0"  iyz="0.0"  izz="0.0" />
+    	</inertial>
     </link>
     <joint name="rear_left_hip_x" type="revolute">
@@ -162,6 +286,17 @@
         <parent link="body" />
         <child link="rear_left_hip" />
+        <dynamics damping="0.1" friction="0.1"/>
         <limit effort="1000" velocity="1000.00" lower="-0.78539816339744827899" upper="0.78539816339744827899" />
     </joint>
+    <transmission name="rear_left_hip_x_trans">
+	  <type>transmission_interface/SimpleTransmission</type>
+	  <joint name="rear_left_hip_x">
+          	<hardwareInterface>hardware_interface/EffortJointInterface</hardwareInterface>
+          </joint>
+	  <actuator name="rear_left_hip_x">
+          	<mechanicalReduction>50</mechanicalReduction>
+          	<hardwareInterface>hardware_interface/EffortJointInterface</hardwareInterface>
+	  </actuator>
+    </transmission>
     <link name="rear_left_upper_leg">
         <visual>
@@ -175,4 +310,8 @@
             </geometry>
         </collision>
+        <inertial>
+           <mass value="1.5" />
+    	   <inertia  ixx="0.0" ixy="0.0"  ixz="0.0"  iyy="0.05"  iyz="0.0"  izz="0.0" />
+    	</inertial>
     </link>
     <joint name="rear_left_hip_y" type="revolute">
@@ -181,6 +320,17 @@
         <parent link="rear_left_hip" />
         <child link="rear_left_upper_leg" />
+        <dynamics damping="0.1" friction="0.1"/>
         <limit effort="1000" velocity="1000.00" lower="-0.89884456477707963539" upper="2.2951079663725435509" />
     </joint>
+    <transmission name="rear_left_hip_y_trans">
+	  <type>transmission_interface/SimpleTransmission</type>
+	  <joint name="rear_left_hip_y">
+          	<hardwareInterface>hardware_interface/EffortJointInterface</hardwareInterface>
+          </joint>
+	  <actuator name="rear_left_hip_y">
+          	<mechanicalReduction>50</mechanicalReduction>
+          	<hardwareInterface>hardware_interface/EffortJointInterface</hardwareInterface>
+	  </actuator>
+    </transmission>
     <link name="rear_left_lower_leg">
         <visual>
@@ -194,4 +344,8 @@
             </geometry>
         </collision>
+        <inertial>
+            <mass value="1.0" />
+    	    <inertia  ixx="0.0" ixy="0.0"  ixz="0.0"  iyy="0.045"  iyz="0.0"  izz="0.0" />
+    	</inertial>
     </link>
     <joint name="rear_left_knee" type="revolute">
@@ -200,6 +354,30 @@
         <parent link="rear_left_upper_leg" />
         <child link="rear_left_lower_leg" />
+        <dynamics damping="0.1" friction="0.1"/>
         <limit effort="1000" velocity="1000.00" lower="-2.7929" upper="-0.267153" />
     </joint>
+     <!-- Contact Sensor -->
+    <gazebo reference="rear_left_lower_leg">
+        <sensor name="rear_left_lower_leg_contactsensor_sensor" type="contact">
+        <always_on>true</always_on>
+        <contact>
+            <collision>rear_left_lower_leg_fixed_joint_lump__rear_bump_sensor_collision</collision>
+        </contact>
+        <plugin filename="libgazebo_ros_bumper.so" name="rear_left_lower_leg_plugin">
+            <bumperTopicName>rear_left_lower_leg_contact</bumperTopicName>
+            <frameName>rear_left_lower_leg</frameName>
+        </plugin>
+        </sensor>
+    </gazebo>
+    <transmission name="rear_left_knee_trans">
+	  <type>transmission_interface/SimpleTransmission</type>
+	  <joint name="rear_left_knee">
+          	<hardwareInterface>hardware_interface/EffortJointInterface</hardwareInterface>
+          </joint>
+	  <actuator name="rear_left_knee">
+          	<mechanicalReduction>50</mechanicalReduction>
+          	<hardwareInterface>hardware_interface/EffortJointInterface</hardwareInterface>
+	  </actuator>
+    </transmission>
     <link name="rear_right_hip">
         <visual>
@@ -213,4 +391,8 @@
             </geometry>
         </collision>
+        <inertial>
+            <mass value="1.5" />
+    	    <inertia  ixx="0.0605" ixy="0.0"  ixz="0.0"  iyy="0.0"  iyz="0.0"  izz="0.0" />
+    	</inertial>
     </link>
     <joint name="rear_right_hip_x" type="revolute">
@@ -219,6 +401,17 @@
         <parent link="body" />
         <child link="rear_right_hip" />
+        <dynamics damping="0.1" friction="0.1"/>
         <limit effort="1000" velocity="1000.00" lower="-0.78539816339744827899" upper="0.78539816339744827899" />
     </joint>
+    <transmission name="rear_right_hip_x_trans">
+	  <type>transmission_interface/SimpleTransmission</type>
+	  <joint name="rear_right_hip_x">
+          	<hardwareInterface>hardware_interface/EffortJointInterface</hardwareInterface>
+          </joint>
+	  <actuator name="rear_right_hip_x">
+          	<mechanicalReduction>50</mechanicalReduction>
+          	<hardwareInterface>hardware_interface/EffortJointInterface</hardwareInterface>
+	  </actuator>
+    </transmission>
     <link name="rear_right_upper_leg">
         <visual>
@@ -232,4 +425,8 @@
             </geometry>
         </collision>
+        <inertial>
+            <mass value="1.5" />
+    	    <inertia  ixx="0.0" ixy="0.0"  ixz="0.0"  iyy="0.05"  iyz="0.0"  izz="0.0" />
+    	</inertial>
     </link>
     <joint name="rear_right_hip_y" type="revolute">
@@ -238,6 +435,17 @@
         <parent link="rear_right_hip" />
         <child link="rear_right_upper_leg" />
+        <dynamics damping="0.1" friction="0.1"/>
         <limit effort="1000" velocity="1000.00" lower="-0.89884456477707963539" upper="2.2951079663725435509" />
     </joint>
+    <transmission name="rear_right_hip_y_trans">
+	  <type>transmission_interface/SimpleTransmission</type>
+	  <joint name="rear_right_hip_y">
+          	<hardwareInterface>hardware_interface/EffortJointInterface</hardwareInterface>
+          </joint>
+	  <actuator name="rear_right_hip_y">
+          	<mechanicalReduction>50</mechanicalReduction>
+          	<hardwareInterface>hardware_interface/EffortJointInterface</hardwareInterface>
+	  </actuator>
+    </transmission>
     <link name="rear_right_lower_leg">
         <visual>
@@ -251,4 +459,8 @@
             </geometry>
         </collision>
+        <inertial>
+            <mass value="1.0" />
+    	    <inertia  ixx="0.0" ixy="0.0"  ixz="0.0"  iyy="0.045"  iyz="0.0"  izz="0.0" />
+    	</inertial>
     </link>
     <joint name="rear_right_knee" type="revolute">
@@ -257,7 +469,36 @@
         <parent link="rear_right_upper_leg" />
         <child link="rear_right_lower_leg" />
+        <dynamics damping="0.1" friction="0.1"/>
         <limit effort="1000" velocity="1000.00" lower="-2.7929" upper="-0.257725" />
     </joint>
+  <!-- Contact Sensor -->
+  <gazebo reference="rear_right_lower_leg">
+    <sensor name="rear_right_lower_leg_contactsensor_sensor" type="contact">
+      <always_on>true</always_on>
+      <contact>
+        <collision>rear_right_lower_leg_fixed_joint_lump__rear_bump_sensor_collision</collision>
+      </contact>
+      <plugin filename="libgazebo_ros_bumper.so" name="rear_right_lower_leg_plugin">
+        <bumperTopicName>rear_right_lower_leg_contact</bumperTopicName>
+        <frameName>rear_right_lower_leg</frameName>
+      </plugin>
+    </sensor>
+  </gazebo>
+    <transmission name="rear_right_knee_trans">
+	  <type>transmission_interface/SimpleTransmission</type>
+	  <joint name="rear_right_knee">
+          	<hardwareInterface>hardware_interface/EffortJointInterface</hardwareInterface>
+          </joint>
+	  <actuator name="rear_right_knee">
+          	<mechanicalReduction>50</mechanicalReduction>
+          	<hardwareInterface>hardware_interface/EffortJointInterface</hardwareInterface>
+	  </actuator>
+    </transmission>
+    <gazebo>
+    	<plugin name="gazebo_ros_control" filename="libgazebo_ros_control.so">
+   	    <!-- <robotNamespace>/spot</robotNamespace> -->
+  	</plugin>
+    </gazebo>
     <!-- Standard accessories. -->
-    <xacro:include filename="$(find spot_gazebo_sim)/urdf/accessories.urdf.xacro" />
+    <!-- <xacro:include filename="$(find spot_gazebo_sim)/urdf/accessories.urdf.xacro" /> -->
 </robot>
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