Commit message: Working version of Spot with ros_control baked in (from different repository).
1. Fixed deprecation notices within spot.urdf.xacro (heavily referenced from clearpath and softserve)
2. Swapped parent / child link on base link to prevent gazebo error.
3. Added inertial components, transmission (ros_control) as well as contact sensors.

File: urdf/spot.urdf.xacro (robot description, xacro)
@@ -1,4 +1,5 @@
 <?xml version="1.0" ?>
 <robot name="spot" xmlns:xacro="http://www.ros.org/wiki/xacro">
+    <link name="base_link"/>
     <link name="body">
         <visual>
@@ -13,9 +14,8 @@
         </collision>
         <inertial>
-             <mass value="16.25" />
-             <inertia  ixx="0.085" ixy="0.0"  ixz="0.0"  iyy="1.045"  iyz="0.0"  izz="1.042" />
-    	</inertial>
-    </link>
-    <link name="base_link"/>
+            <mass value="16.25" />
+            <inertia  ixx="0.085" ixy="0.0"  ixz="0.0"  iyy="1.045"  iyz="0.0"  izz="1.042" />
+        </inertial>
+    </link>
     <joint name="base_link_joint" type="fixed">
         <origin xyz="0 0 0" rpy="0 0 0" />
@@ -48,6 +48,6 @@
         <inertial>
             <mass value="1.5" />
-    	    <inertia  ixx="0.0605" ixy="0.0"  ixz="0.0"  iyy="0.0"  iyz="0.0"  izz="0.0" />
-    	</inertial>
+            <inertia  ixx="0.0605" ixy="0.0"  ixz="0.0"  iyy="0.0"  iyz="0.0"  izz="0.0" />
+        </inertial>
     </link>
     <joint name="front_left_hip_x" type="revolute">
@@ -56,16 +56,16 @@
         <parent link="body" />
         <child link="front_left_hip" />
-	    <dynamics damping="0.1" friction="0.1"/>
+        <dynamics damping="0.1" friction="0.1"/>
         <limit effort="1000" velocity="1000.00" lower="-0.78539816339744827899" upper="0.78539816339744827899" />
     </joint>
     <transmission name="front_left_hip_x_trans">
-	  <type>transmission_interface/SimpleTransmission</type>
-	  <joint name="front_left_hip_x">
-          	<hardwareInterface>hardware_interface/EffortJointInterface</hardwareInterface>
-          </joint>
-	  <actuator name="front_left_hip_x">
-          	<mechanicalReduction>50</mechanicalReduction>
-          	<hardwareInterface>hardware_interface/EffortJointInterface</hardwareInterface>
-	  </actuator>
+        <type>transmission_interface/SimpleTransmission</type>
+        <joint name="front_left_hip_x">
+            <hardwareInterface>hardware_interface/EffortJointInterface</hardwareInterface>
+        </joint>
+        <actuator name="front_left_hip_x">
+            <mechanicalReduction>50</mechanicalReduction>
+            <hardwareInterface>hardware_interface/EffortJointInterface</hardwareInterface>
+        </actuator>
     </transmission>
     <link name="front_left_upper_leg">
@@ -82,6 +82,6 @@
         <inertial>
             <mass value="1.5" />
-    	    <inertia  ixx="0.0" ixy="0.0"  ixz="0.0"  iyy="0.05"  iyz="0.0"  izz="0.0" />
-    	</inertial>
+            <inertia  ixx="0.0" ixy="0.0"  ixz="0.0"  iyy="0.05"  iyz="0.0"  izz="0.0" />
+        </inertial>
     </link>
     <joint name="front_left_hip_y" type="revolute">
@@ -90,16 +90,16 @@
         <parent link="front_left_hip" />
         <child link="front_left_upper_leg" />
-	    <dynamics damping="0.1" friction="0.1"/>
+        <dynamics damping="0.1" friction="0.1"/>
         <limit effort="1000" velocity="1000.00" lower="-0.89884456477707963539" upper="2.2951079663725435509" />
     </joint>
     <transmission name="front_left_hip_y_trans">
-	  <type>transmission_interface/SimpleTransmission</type>
-	  <joint name="front_left_hip_y">
-          	<hardwareInterface>hardware_interface/EffortJointInterface</hardwareInterface>
-          </joint>
-	  <actuator name="front_left_hip_y">
-          	<mechanicalReduction>50</mechanicalReduction>
-          	<hardwareInterface>hardware_interface/EffortJointInterface</hardwareInterface>
-	  </actuator>
+        <type>transmission_interface/SimpleTransmission</type>
+        <joint name="front_left_hip_y">
+            <hardwareInterface>hardware_interface/EffortJointInterface</hardwareInterface>
+        </joint>
+        <actuator name="front_left_hip_y">
+            <mechanicalReduction>50</mechanicalReduction>
+            <hardwareInterface>hardware_interface/EffortJointInterface</hardwareInterface>
+        </actuator>
     </transmission>
     <link name="front_left_lower_leg">
@@ -116,6 +116,6 @@
         <inertial>right
             <mass value="1.0" />
-    	    <inertia  ixx="0.0" ixy="0.0"  ixz="0.0"  iyy="0.045"  iyz="0.0"  izz="0.0" />
-    	</inertial>
+            <inertia  ixx="0.0" ixy="0.0"  ixz="0.0"  iyy="0.045"  iyz="0.0"  izz="0.0" />
+        </inertial>
     </link>
     <joint name="front_left_knee" type="revolute">
@@ -127,5 +127,5 @@
         <limit effort="1000" velocity="1000.00" lower="-2.7929" upper="-0.254801" />
     </joint>
-    <!-- Optional Contact Sensor (SoftServeSAG) -->
+    <!-- Contact Sensor -->
     <gazebo reference="front_left_lower_leg">
         <sensor name="front_left_lower_leg_contactsensor_sensor" type="contact">
@@ -141,12 +141,12 @@
     </gazebo>
     <transmission name="front_left_knee_trans">
-	  <type>transmission_interface/SimpleTransmission</type>
-	  <joint name="front_left_knee">
-          	<hardwareInterface>hardware_interface/EffortJointInterface</hardwareInterface>
-          </joint>
-	  <actuator name="front_left_knee">
-          	<mechanicalReduction>50</mechanicalReduction>
-          	<hardwareInterface>hardware_interface/EffortJointInterface</hardwareInterface>
-	  </actuator>
+        <type>transmission_interface/SimpleTransmission</type>
+        <joint name="front_left_knee">
+            <hardwareInterface>hardware_interface/EffortJointInterface</hardwareInterface>
+        </joint>
+		<actuator name="front_left_knee">
+            <mechanicalReduction>50</mechanicalReduction>
+            <hardwareInterface>hardware_interface/EffortJointInterface</hardwareInterface>
+        </actuator>
     </transmission>
     <link name="front_right_hip">
@@ -163,6 +163,6 @@
         <inertial>
             <mass value="1.5" />
-    	    <inertia  ixx="0.0605" ixy="0.0"  ixz="0.0"  iyy="0.0"  iyz="0.0"  izz="0.0" />
-    	</inertial>
+            <inertia  ixx="0.0605" ixy="0.0"  ixz="0.0"  iyy="0.0"  iyz="0.0"  izz="0.0" />
+        </inertial>
     </link>
     <joint name="front_right_hip_x" type="revolute">
@@ -175,12 +175,12 @@
     </joint>
     <transmission name="front_right_hip_x_trans">
-	  <type>transmission_interface/SimpleTransmission</type>
-	  <joint name="front_right_hip_x">
-          	<hardwareInterface>hardware_interface/EffortJointInterface</hardwareInterface>
-          </joint>
-	  <actuator name="front_right_hip_x">
-          	<mechanicalReduction>50</mechanicalReduction>
-          	<hardwareInterface>hardware_interface/EffortJointInterface</hardwareInterface>
-	  </actuator>
+        <type>transmission_interface/SimpleTransmission</type>
+        <joint name="front_right_hip_x">
+            <hardwareInterface>hardware_interface/EffortJointInterface</hardwareInterface>
+        </joint>
+		<actuator name="front_right_hip_x">
+            <mechanicalReduction>50</mechanicalReduction>
+            <hardwareInterface>hardware_interface/EffortJointInterface</hardwareInterface>
+      	</actuator>
     </transmission>
     <link name="front_right_upper_leg">
@@ -197,6 +197,6 @@
         <inertial>
             <mass value="1.5" />
-    	    <inertia  ixx="0.0" ixy="0.0"  ixz="0.0"  iyy="0.05"  iyz="0.0"  izz="0.0" />
-    	</inertial>
+            <inertia  ixx="0.0" ixy="0.0"  ixz="0.0"  iyy="0.05"  iyz="0.0"  izz="0.0" />
+        </inertial>
     </link>
     <joint name="front_right_hip_y" type="revolute">
@@ -209,12 +209,12 @@
     </joint>
     <transmission name="front_right_hip_y_trans">
-	  <type>transmission_interface/SimpleTransmission</type>
-	  <joint name="front_right_hip_y">
-          	<hardwareInterface>hardware_interface/EffortJointInterface</hardwareInterface>
-          </joint>
-	  <actuator name="front_right_hip_y">
-          	<mechanicalReduction>50</mechanicalReduction>
-          	<hardwareInterface>hardware_interface/EffortJointInterface</hardwareInterface>
-	  </actuator>
+        <type>transmission_interface/SimpleTransmission</type>
+        <joint name="front_right_hip_y">
+            <hardwareInterface>hardware_interface/EffortJointInterface</hardwareInterface>
+        </joint>
+        <actuator name="front_right_hip_y">
+            <mechanicalReduction>50</mechanicalReduction>
+            <hardwareInterface>hardware_interface/EffortJointInterface</hardwareInterface>
+        </actuator>
     </transmission>
     <link name="front_right_lower_leg">
@@ -231,6 +231,6 @@
         <inertial>
             <mass value="1.0" />
-    	    <inertia  ixx="0.0" ixy="0.0"  ixz="0.0"  iyy="0.045"  iyz="0.0"  izz="0.0" />
-    	</inertial>
+            <inertia  ixx="0.0" ixy="0.0"  ixz="0.0"  iyy="0.045"  iyz="0.0"  izz="0.0" />
+        </inertial>
     </link>
     <joint name="front_right_knee" type="revolute">
@@ -256,12 +256,12 @@
     </gazebo>
     <transmission name="front_right_knee_trans">
-	  <type>transmission_interface/SimpleTransmission</type>
-	  <joint name="front_right_knee">
-          	<hardwareInterface>hardware_interface/EffortJointInterface</hardwareInterface>
-          </joint>
-	  <actuator name="front_right_knee">
-          	<mechanicalReduction>50</mechanicalReduction>
-          	<hardwareInterface>hardware_interface/EffortJointInterface</hardwareInterface>
-	  </actuator>
+        <type>transmission_interface/SimpleTransmission</type>
+        <joint name="front_right_knee">
+            <hardwareInterface>hardware_interface/EffortJointInterface</hardwareInterface>
+        </joint>
+        <actuator name="front_right_knee">
+            <mechanicalReduction>50</mechanicalReduction>
+            <hardwareInterface>hardware_interface/EffortJointInterface</hardwareInterface>
+        </actuator>
     </transmission>
     <link name="rear_left_hip">
@@ -278,6 +278,6 @@
         <inertial>
             <mass value="1.5" />
-    	    <inertia  ixx="0.0605" ixy="0.0"  ixz="0.0"  iyy="0.0"  iyz="0.0"  izz="0.0" />
-    	</inertial>
+            <inertia  ixx="0.0605" ixy="0.0"  ixz="0.0"  iyy="0.0"  iyz="0.0"  izz="0.0" />
+        </inertial>
     </link>
     <joint name="rear_left_hip_x" type="revolute">
@@ -290,12 +290,12 @@
     </joint>
     <transmission name="rear_left_hip_x_trans">
-	  <type>transmission_interface/SimpleTransmission</type>
-	  <joint name="rear_left_hip_x">
-          	<hardwareInterface>hardware_interface/EffortJointInterface</hardwareInterface>
-          </joint>
-	  <actuator name="rear_left_hip_x">
-          	<mechanicalReduction>50</mechanicalReduction>
-          	<hardwareInterface>hardware_interface/EffortJointInterface</hardwareInterface>
-	  </actuator>
+        <type>transmission_interface/SimpleTransmission</type>
+        <joint name="rear_left_hip_x">
+            <hardwareInterface>hardware_interface/EffortJointInterface</hardwareInterface>
+        </joint>
+        <actuator name="rear_left_hip_x">
+            <mechanicalReduction>50</mechanicalReduction>
+            <hardwareInterface>hardware_interface/EffortJointInterface</hardwareInterface>
+        </actuator>
     </transmission>
     <link name="rear_left_upper_leg">
@@ -312,6 +312,6 @@
         <inertial>
            <mass value="1.5" />
-    	   <inertia  ixx="0.0" ixy="0.0"  ixz="0.0"  iyy="0.05"  iyz="0.0"  izz="0.0" />
-    	</inertial>
+           <inertia  ixx="0.0" ixy="0.0"  ixz="0.0"  iyy="0.05"  iyz="0.0"  izz="0.0" />
+        </inertial>
     </link>
     <joint name="rear_left_hip_y" type="revolute">
@@ -324,12 +324,12 @@
     </joint>
     <transmission name="rear_left_hip_y_trans">
-	  <type>transmission_interface/SimpleTransmission</type>
-	  <joint name="rear_left_hip_y">
-          	<hardwareInterface>hardware_interface/EffortJointInterface</hardwareInterface>
-          </joint>
-	  <actuator name="rear_left_hip_y">
-          	<mechanicalReduction>50</mechanicalReduction>
-          	<hardwareInterface>hardware_interface/EffortJointInterface</hardwareInterface>
-	  </actuator>
+        <type>transmission_interface/SimpleTransmission</type>
+        <joint name="rear_left_hip_y">
+            <hardwareInterface>hardware_interface/EffortJointInterface</hardwareInterface>
+        </joint>
+        <actuator name="rear_left_hip_y">
+            <mechanicalReduction>50</mechanicalReduction>
+            <hardwareInterface>hardware_interface/EffortJointInterface</hardwareInterface>
+        </actuator>
     </transmission>
     <link name="rear_left_lower_leg">
@@ -346,6 +346,6 @@
         <inertial>
             <mass value="1.0" />
-    	    <inertia  ixx="0.0" ixy="0.0"  ixz="0.0"  iyy="0.045"  iyz="0.0"  izz="0.0" />
-    	</inertial>
+            <inertia  ixx="0.0" ixy="0.0"  ixz="0.0"  iyy="0.045"  iyz="0.0"  izz="0.0" />
+        </inertial>
     </link>
     <joint name="rear_left_knee" type="revolute">
@@ -371,12 +371,12 @@
     </gazebo>
     <transmission name="rear_left_knee_trans">
-	  <type>transmission_interface/SimpleTransmission</type>
-	  <joint name="rear_left_knee">
-          	<hardwareInterface>hardware_interface/EffortJointInterface</hardwareInterface>
-          </joint>
-	  <actuator name="rear_left_knee">
-          	<mechanicalReduction>50</mechanicalReduction>
-          	<hardwareInterface>hardware_interface/EffortJointInterface</hardwareInterface>
-	  </actuator>
+        <type>transmission_interface/SimpleTransmission</type>
+        <joint name="rear_left_knee">
+            <hardwareInterface>hardware_interface/EffortJointInterface</hardwareInterface>
+        </joint>
+        <actuator name="rear_left_knee">
+            <mechanicalReduction>50</mechanicalReduction>
+            <hardwareInterface>hardware_interface/EffortJointInterface</hardwareInterface>
+        </actuator>
     </transmission>
     <link name="rear_right_hip">
@@ -393,6 +393,6 @@
         <inertial>
             <mass value="1.5" />
-    	    <inertia  ixx="0.0605" ixy="0.0"  ixz="0.0"  iyy="0.0"  iyz="0.0"  izz="0.0" />
-    	</inertial>
+            <inertia  ixx="0.0605" ixy="0.0"  ixz="0.0"  iyy="0.0"  iyz="0.0"  izz="0.0" />
+        </inertial>
     </link>
     <joint name="rear_right_hip_x" type="revolute">
@@ -405,12 +405,12 @@
     </joint>
     <transmission name="rear_right_hip_x_trans">
-	  <type>transmission_interface/SimpleTransmission</type>
-	  <joint name="rear_right_hip_x">
-          	<hardwareInterface>hardware_interface/EffortJointInterface</hardwareInterface>
-          </joint>
-	  <actuator name="rear_right_hip_x">
-          	<mechanicalReduction>50</mechanicalReduction>
-          	<hardwareInterface>hardware_interface/EffortJointInterface</hardwareInterface>
-	  </actuator>
+        <type>transmission_interface/SimpleTransmission</type>
+        <joint name="rear_right_hip_x">
+            <hardwareInterface>hardware_interface/EffortJointInterface</hardwareInterface>
+        </joint>
+        <actuator name="rear_right_hip_x">
+            <mechanicalReduction>50</mechanicalReduction>
+            <hardwareInterface>hardware_interface/EffortJointInterface</hardwareInterface>
+        </actuator>
     </transmission>
     <link name="rear_right_upper_leg">
@@ -427,6 +427,6 @@
         <inertial>
             <mass value="1.5" />
-    	    <inertia  ixx="0.0" ixy="0.0"  ixz="0.0"  iyy="0.05"  iyz="0.0"  izz="0.0" />
-    	</inertial>
+            <inertia  ixx="0.0" ixy="0.0"  ixz="0.0"  iyy="0.05"  iyz="0.0"  izz="0.0" />
+        </inertial>
     </link>
     <joint name="rear_right_hip_y" type="revolute">
@@ -439,12 +439,12 @@
     </joint>
     <transmission name="rear_right_hip_y_trans">
-	  <type>transmission_interface/SimpleTransmission</type>
-	  <joint name="rear_right_hip_y">
-          	<hardwareInterface>hardware_interface/EffortJointInterface</hardwareInterface>
-          </joint>
-	  <actuator name="rear_right_hip_y">
-          	<mechanicalReduction>50</mechanicalReduction>
-          	<hardwareInterface>hardware_interface/EffortJointInterface</hardwareInterface>
-	  </actuator>
+        <type>transmission_interface/SimpleTransmission</type>
+        <joint name="rear_right_hip_y">
+            <hardwareInterface>hardware_interface/EffortJointInterface</hardwareInterface>
+        </joint>
+        <actuator name="rear_right_hip_y">
+            <mechanicalReduction>50</mechanicalReduction>
+            <hardwareInterface>hardware_interface/EffortJointInterface</hardwareInterface>
+        </actuator>
     </transmission>
     <link name="rear_right_lower_leg">
@@ -461,6 +461,6 @@
         <inertial>
             <mass value="1.0" />
-    	    <inertia  ixx="0.0" ixy="0.0"  ixz="0.0"  iyy="0.045"  iyz="0.0"  izz="0.0" />
-    	</inertial>
+            <inertia  ixx="0.0" ixy="0.0"  ixz="0.0"  iyy="0.045"  iyz="0.0"  izz="0.0" />
+        </inertial>
     </link>
     <joint name="rear_right_knee" type="revolute">
@@ -472,31 +472,31 @@
         <limit effort="1000" velocity="1000.00" lower="-2.7929" upper="-0.257725" />
     </joint>
-  <!-- Contact Sensor -->
-  <gazebo reference="rear_right_lower_leg">
-    <sensor name="rear_right_lower_leg_contactsensor_sensor" type="contact">
-      <always_on>true</always_on>
-      <contact>
-        <collision>rear_right_lower_leg_fixed_joint_lump__rear_bump_sensor_collision</collision>
-      </contact>
-      <plugin filename="libgazebo_ros_bumper.so" name="rear_right_lower_leg_plugin">
-        <bumperTopicName>rear_right_lower_leg_contact</bumperTopicName>
-        <frameName>rear_right_lower_leg</frameName>
-      </plugin>
-    </sensor>
-  </gazebo>
+    <!-- Contact Sensor -->
+    <gazebo reference="rear_right_lower_leg">
+        <sensor name="rear_right_lower_leg_contactsensor_sensor" type="contact">
+            <always_on>true</always_on>
+            <contact>
+                <collision>rear_right_lower_leg_fixed_joint_lump__rear_bump_sensor_collision</collision>
+            </contact>
+            <plugin filename="libgazebo_ros_bumper.so" name="rear_right_lower_leg_plugin">
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